File: hardware/perpheral/p2hex-001.sch (EAGLE design)
At the start: 2 parts

Commit message: First try.
Parts:
- added S1, S2: (no value), switch-dil:A1353HEX
Connections:
- new net ANLG0: JP1.3, S2.1
- new net ANLG1: JP1.7, S2.4
- new net ANLG2: JP1.11, S2.8
- new net ANLG3: JP1.15, S2.2
- new net DTCT0: JP1.2, S1.1
- new net DTCT1: JP1.6, S1.4
- new net DTCT2: JP1.10, S1.8
- new net DTCT3: JP1.14, S1.2
- new net GND: JP1.1, JP1.13, JP1.5, JP1.9, S1.C
- new net VCC: JP1.12, JP1.16, JP1.4, JP1.8, S2.C
Other:
- note added: "GeekPort II 1: GND 2: DTCT0 3: ANLG0 4: Vcc/2"
- note added: "Pineapple -> Switch 1->1 2->4 4->8 8->2"
- moved on the sheet: JP1

Commit message: Second try.
Parts:
- added U$1: PINEAPPLE450_SILK, pineapple:PINEAPPLE450_SILK
Changed lines of the file:
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@@
 <part name="SUPPLY3" library="supply2" library_urn="urn:adsk.eagle:library:372" deviceset="VCC" device=""/>
 <part name="SUPPLY4" library="supply2" library_urn="urn:adsk.eagle:library:372" deviceset="VCC" device=""/>
+<part name="U$1" library="pineapple" deviceset="PINEAPPLE450_SILK" device=""/>
 </parts>
 <sheets>
@@
 <attribute name="VALUE" x="59.055" y="120.015" size="1.778" layer="96"/>
 </instance>
+<instance part="U$1" gate="G$1" x="241.3" y="142.24" smashed="yes"/>
 </instances>
 <busses>
