File: hardware/perpheral/p2hex-001.brd (EAGLE design)
At the start: 89 x 51 mm, 2 parts

Commit message: First try.
Parts:
- added S1, S2: (no value), switch-dil:A1353HEX
- moved LOGO1 23.1 mm to (5.00, 21.0), flipped to the bottom
- moved JP1 10.2 mm to (13.0, 15.5)
Connections:
- new net ANLG0: JP1.3, S2.1
- new net ANLG1: JP1.7, S2.4
- new net ANLG2: JP1.11, S2.8
- new net ANLG3: JP1.15, S2.2
- new net DTCT0: JP1.2, S1.1
- new net DTCT1: JP1.6, S1.4
- new net DTCT2: JP1.10, S1.8
- new net DTCT3: JP1.14, S1.2
- new net GND: JP1.1, JP1.13, JP1.5, JP1.9, S1.C
- new net VCC: JP1.12, JP1.16, JP1.4, JP1.8, S2.C
Routing:
- net GND: track 0.00 -> 32.4 mm
- net VCC: track 0.00 -> 31.7 mm
- net ANLG0: track 0.00 -> 23.2 mm
- net DTCT3: track 0.00 -> 22.2 mm
- net ANLG1: track 0.00 -> 17.1 mm
- net ANLG3: track 0.00 -> 14.8 mm
- net DTCT2: track 0.00 -> 12.4 mm
- net DTCT1: track 0.00 -> 11.4 mm
- net DTCT0: track 0.00 -> 8.95 mm
- net ANLG2: track 0.00 -> 7.60 mm
Other:
- board size 89 x 51 mm -> 18 x 31 mm
- board text added: "2"
- board text added: "4"
- board text added: "8"

Commit message: Second try.
Parts:
- added U$1: PINEAPPLE450_SILK, pineapple:PINEAPPLE450_SILK
- moved LOGO1 11.0 mm to (5.00, 10.0), turned to 90 degrees
Routing:
- net GND: track 32.4 -> 28.5 mm
- net ANLG0: track 23.2 -> 19.9 mm
- net DTCT2: track 12.4 -> 15.0 mm
- net DTCT3: track 22.2 -> 20.4 mm
- net DTCT1: track 11.4 -> 10.1 mm
- net ANLG1: track 17.1 -> 16.4 mm
- added copper zone on layer 1, net GND
- added copper zone on layer 16, net GND
Other:
- board text added: "Hex Sw 0.0.1-X"
- board text removed: "2"
- board text removed: "4"
- board text removed: "8"

Commit message: Moved Pineapple logo.
Parts:
- moved U$1 11.0 mm to (0.50, 21.0)
Changed lines of the file:
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@@
 <layer number="19" name="Unrouted" color="6" fill="1" visible="yes" active="yes"/>
 <layer number="20" name="Dimension" color="24" fill="1" visible="yes" active="yes"/>
-<layer number="21" name="tPlace" color="7" fill="1" visible="yes" active="yes"/>
-<layer number="22" name="bPlace" color="7" fill="1" visible="no" active="yes"/>
+<layer number="21" name="tPlace" color="7" fill="1" visible="no" active="yes"/>
+<layer number="22" name="bPlace" color="7" fill="1" visible="yes" active="yes"/>
 <layer number="23" name="tOrigins" color="15" fill="1" visible="yes" active="yes"/>
 <layer number="24" name="bOrigins" color="15" fill="1" visible="yes" active="yes"/>
-<layer number="25" name="tNames" color="7" fill="1" visible="yes" active="yes"/>
-<layer number="26" name="bNames" color="7" fill="1" visible="no" active="yes"/>
+<layer number="25" name="tNames" color="7" fill="1" visible="no" active="yes"/>
+<layer number="26" name="bNames" color="7" fill="1" visible="yes" active="yes"/>
 <layer number="27" name="tValues" color="7" fill="1" visible="no" active="yes"/>
 <layer number="28" name="bValues" color="7" fill="1" visible="no" active="yes"/>
@@
 <attribute name="VALUE" x="11.731" y="15.92" size="1.27" layer="27" ratio="10" rot="R90"/>
 </element>
-<element name="U$1" library="pineapple" package="PINEAPPLE450_SILK" value="PINEAPPLE450_SILK" x="0.5" y="10" smashed="yes" rot="MR90"/>
+<element name="U$1" library="pineapple" package="PINEAPPLE450_SILK" value="PINEAPPLE450_SILK" x="0.5" y="21" smashed="yes" rot="MR90"/>
 </elements>
 <signals>
