File: hardware/peripheral/p2hex-001.brd (EAGLE design)
At the start: 18 x 31 mm, 5 parts

Commit message: Silk.
Parts:
- renumbered S1 to S1C, S2 to S2R
Changed lines of the file:
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@@
 <layer number="19" name="Unrouted" color="6" fill="1" visible="yes" active="yes"/>
 <layer number="20" name="Dimension" color="24" fill="1" visible="yes" active="yes"/>
-<layer number="21" name="tPlace" color="7" fill="1" visible="no" active="yes"/>
-<layer number="22" name="bPlace" color="7" fill="1" visible="yes" active="yes"/>
+<layer number="21" name="tPlace" color="7" fill="1" visible="yes" active="yes"/>
+<layer number="22" name="bPlace" color="7" fill="1" visible="no" active="yes"/>
 <layer number="23" name="tOrigins" color="15" fill="1" visible="yes" active="yes"/>
 <layer number="24" name="bOrigins" color="15" fill="1" visible="yes" active="yes"/>
-<layer number="25" name="tNames" color="7" fill="1" visible="no" active="yes"/>
-<layer number="26" name="bNames" color="7" fill="1" visible="yes" active="yes"/>
+<layer number="25" name="tNames" color="7" fill="1" visible="yes" active="yes"/>
+<layer number="26" name="bNames" color="7" fill="1" visible="no" active="yes"/>
 <layer number="27" name="tValues" color="7" fill="1" visible="no" active="yes"/>
 <layer number="28" name="bValues" color="7" fill="1" visible="no" active="yes"/>
@@
 <attribute name="VALUE" x="17.445" y="5.34" size="1.27" layer="27" rot="R90"/>
 </element>
-<element name="S1" library="switch-dil" library_urn="urn:adsk.eagle:library:375" package="A1353HEX" package3d_urn="urn:adsk.eagle:package:27207/1" value="" x="5" y="10" smashed="yes" rot="R90">
+<element name="S1C" library="switch-dil" library_urn="urn:adsk.eagle:library:375" package="A1353HEX" package3d_urn="urn:adsk.eagle:package:27207/1" value="" x="5" y="10" smashed="yes" rot="R90">
 <attribute name="MF" value="" x="5" y="10" size="1.778" layer="27" rot="R90" display="off"/>
 <attribute name="MPN" value="" x="5" y="10" size="1.778" layer="27" rot="R90" display="off"/>
-<attribute name="NAME" x="0.5" y="4" size="1" layer="25" ratio="10" rot="R90" align="top-center"/>
+<attribute name="NAME" x="0.5" y="3" size="1" layer="25" ratio="10" rot="R90" align="top-center"/>
 <attribute name="OC_FARNELL" value="unknown" x="5" y="10" size="1.778" layer="27" rot="R90" display="off"/>
 <attribute name="OC_NEWARK" value="unknown" x="5" y="10" size="1.778" layer="27" rot="R90" display="off"/>
 <attribute name="VALUE" x="11.731" y="4.92" size="1.27" layer="27" ratio="10" rot="R90"/>
 </element>
-<element name="S2" library="switch-dil" library_urn="urn:adsk.eagle:library:375" package="A1353HEX" package3d_urn="urn:adsk.eagle:package:27207/1" value="" x="5" y="21" smashed="yes" rot="R90">
+<element name="S2R" library="switch-dil" library_urn="urn:adsk.eagle:library:375" package="A1353HEX" package3d_urn="urn:adsk.eagle:package:27207/1" value="" x="5" y="21" smashed="yes" rot="R90">
 <attribute name="MF" value="" x="5" y="21" size="1.778" layer="27" rot="R90" display="off"/>
 <attribute name="MPN" value="" x="5" y="21" size="1.778" layer="27" rot="R90" display="off"/>
-<attribute name="NAME" x="0.5" y="27" size="1" layer="25" ratio="10" rot="R90" align="top-center"/>
+<attribute name="NAME" x="0.5" y="28" size="1" layer="25" ratio="10" rot="R90" align="top-center"/>
 <attribute name="OC_FARNELL" value="unknown" x="5" y="21" size="1.778" layer="27" rot="R90" display="off"/>
 <attribute name="OC_NEWARK" value="unknown" x="5" y="21" size="1.778" layer="27" rot="R90" display="off"/>
@@
 <signal name="GND">
 <contactref element="JP1" pad="1"/>
-<contactref element="S1" pad="C"/>
+<contactref element="S1C" pad="C"/>
 <contactref element="JP1" pad="5"/>
 <contactref element="JP1" pad="9"/>
@@
 <signal name="DTCT0">
 <contactref element="JP1" pad="2"/>
-<contactref element="S1" pad="1"/>
+<contactref element="S1C" pad="1"/>
 <wire x1="7.62" y1="10.668" x2="7.62" y2="13.716" width="0.1524" layer="1"/>
 <wire x1="11.5824" y1="6.7056" x2="7.62" y2="10.668" width="0.1524" layer="1"/>
@@
 <contactref element="JP1" pad="12"/>
 <contactref element="JP1" pad="8"/>
-<contactref element="S2" pad="C"/>
+<contactref element="S2R" pad="C"/>
 <wire x1="11.5824" y1="10.3632" x2="11.5824" y2="9.2964" width="0.1524" layer="1"/>
 <wire x1="10.668" y1="11.2776" x2="11.5824" y2="10.3632" width="0.1524" layer="1"/>
@@
 <signal name="DTCT1">
 <contactref element="JP1" pad="6"/>
-<contactref element="S1" pad="4"/>
+<contactref element="S1C" pad="4"/>
 <wire x1="3.048" y1="13.716" x2="2.5908" y2="13.716" width="0.1524" layer="16"/>
 <wire x1="4.8768" y1="11.8872" x2="3.048" y2="13.716" width="0.1524" layer="16"/>
@@
 <signal name="DTCT2">
 <contactref element="JP1" pad="10"/>
-<contactref element="S1" pad="8"/>
+<contactref element="S1C" pad="8"/>
 <wire x1="7.4676" y1="10.3632" x2="7.4676" y2="6.2484" width="0.1524" layer="1"/>
 <wire x1="6.5532" y1="11.2776" x2="7.4676" y2="10.3632" width="0.1524" layer="1"/>
@@
 <signal name="DTCT3">
 <contactref element="JP1" pad="14"/>
-<contactref element="S1" pad="2"/>
+<contactref element="S1C" pad="2"/>
 <wire x1="2.5908" y1="9.4488" x2="2.5908" y2="6.2484" width="0.1524" layer="1"/>
 <wire x1="6.2484" y1="13.1064" x2="2.5908" y2="9.4488" width="0.1524" layer="1"/>
@@
 <signal name="ANLG0">
 <contactref element="JP1" pad="3"/>
-<contactref element="S2" pad="1"/>
+<contactref element="S2R" pad="1"/>
 <wire x1="7.62" y1="21.9456" x2="7.62" y2="24.6888" width="0.1524" layer="16"/>
 <wire x1="11.7348" y1="17.8308" x2="7.62" y2="21.9456" width="0.1524" layer="16"/>
@@
 <signal name="ANLG1">
 <contactref element="JP1" pad="7"/>
-<contactref element="S2" pad="4"/>
+<contactref element="S2R" pad="4"/>
 <wire x1="2.5908" y1="24.384" x2="2.5908" y2="24.6888" width="0.1524" layer="16"/>
 <wire x1="11.7348" y1="15.24" x2="2.5908" y2="24.384" width="0.1524" layer="16"/>
@@
 </signal>
 <signal name="ANLG3">
-<contactref element="S2" pad="2"/>
+<contactref element="S2R" pad="2"/>
 <contactref element="JP1" pad="15"/>
 <wire x1="5.1816" y1="17.2212" x2="2.5908" y2="17.2212" width="0.1524" layer="1"/>
@@
 </signal>
 <signal name="ANLG2">
-<contactref element="S2" pad="8"/>
+<contactref element="S2R" pad="8"/>
 <contactref element="JP1" pad="11"/>
 <wire x1="10.668" y1="17.2212" x2="7.62" y2="17.2212" width="0.1524" layer="1"/>
