File: hardware/peripheral/p2hex-001.brd (EAGLE design)
At the start: 18 x 31 mm, 5 parts

Commit message: Silk.
Parts:
- renumbered JP1 to SV1
Changed lines of the file:
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@@
 <elements>
 <element name="LOGO1" library="SparkFun-Aesthetics" package="OSHW-LOGO-S_COPPER" value="OSHW-LOGOS-COPPER" x="5" y="10" smashed="yes" rot="MR90"/>
-<element name="JP1" library="pinhead" library_urn="urn:adsk.eagle:library:325" package="2X08" package3d_urn="urn:adsk.eagle:package:22481/2" value="" x="13" y="15.5" smashed="yes" rot="R90">
+<element name="SV1" library="pinhead" library_urn="urn:adsk.eagle:library:325" package="2X08" package3d_urn="urn:adsk.eagle:package:22481/2" value="" x="13" y="15.5" smashed="yes" rot="R90">
 <attribute name="NAME" x="18.5" y="15.5" size="1" layer="25" ratio="10" rot="R90" align="top-center"/>
 <attribute name="POPULARITY" value="6" x="13" y="15.5" size="1.778" layer="27" rot="R90" display="off"/>
@@
 <signals>
 <signal name="GND">
-<contactref element="JP1" pad="1"/>
+<contactref element="SV1" pad="1"/>
 <contactref element="S1C" pad="C"/>
-<contactref element="JP1" pad="5"/>
-<contactref element="JP1" pad="9"/>
-<contactref element="JP1" pad="13"/>
+<contactref element="SV1" pad="5"/>
+<contactref element="SV1" pad="9"/>
+<contactref element="SV1" pad="13"/>
 <wire x1="14.1732" y1="17.9832" x2="14.1732" y2="16.9164" width="0.1524" layer="16"/>
 <wire x1="13.2588" y1="18.8976" x2="14.1732" y2="17.9832" width="0.1524" layer="16"/>
@@
 </signal>
 <signal name="DTCT0">
-<contactref element="JP1" pad="2"/>
+<contactref element="SV1" pad="2"/>
 <contactref element="S1C" pad="1"/>
 <wire x1="7.62" y1="10.668" x2="7.62" y2="13.716" width="0.1524" layer="1"/>
@@
 </signal>
 <signal name="VCC">
-<contactref element="JP1" pad="4"/>
-<contactref element="JP1" pad="16"/>
-<contactref element="JP1" pad="12"/>
-<contactref element="JP1" pad="8"/>
+<contactref element="SV1" pad="4"/>
+<contactref element="SV1" pad="16"/>
+<contactref element="SV1" pad="12"/>
+<contactref element="SV1" pad="8"/>
 <contactref element="S2R" pad="C"/>
 <wire x1="11.5824" y1="10.3632" x2="11.5824" y2="9.2964" width="0.1524" layer="1"/>
@@
 </signal>
 <signal name="DTCT1">
-<contactref element="JP1" pad="6"/>
+<contactref element="SV1" pad="6"/>
 <contactref element="S1C" pad="4"/>
 <wire x1="3.048" y1="13.716" x2="2.5908" y2="13.716" width="0.1524" layer="16"/>
@@
 </signal>
 <signal name="DTCT2">
-<contactref element="JP1" pad="10"/>
+<contactref element="SV1" pad="10"/>
 <contactref element="S1C" pad="8"/>
 <wire x1="7.4676" y1="10.3632" x2="7.4676" y2="6.2484" width="0.1524" layer="1"/>
@@
 </signal>
 <signal name="DTCT3">
-<contactref element="JP1" pad="14"/>
+<contactref element="SV1" pad="14"/>
 <contactref element="S1C" pad="2"/>
 <wire x1="2.5908" y1="9.4488" x2="2.5908" y2="6.2484" width="0.1524" layer="1"/>
@@
 </signal>
 <signal name="ANLG0">
-<contactref element="JP1" pad="3"/>
+<contactref element="SV1" pad="3"/>
 <contactref element="S2R" pad="1"/>
 <wire x1="7.62" y1="21.9456" x2="7.62" y2="24.6888" width="0.1524" layer="16"/>
@@
 </signal>
 <signal name="ANLG1">
-<contactref element="JP1" pad="7"/>
+<contactref element="SV1" pad="7"/>
 <contactref element="S2R" pad="4"/>
 <wire x1="2.5908" y1="24.384" x2="2.5908" y2="24.6888" width="0.1524" layer="16"/>
@@
 <signal name="ANLG3">
 <contactref element="S2R" pad="2"/>
-<contactref element="JP1" pad="15"/>
+<contactref element="SV1" pad="15"/>
 <wire x1="5.1816" y1="17.2212" x2="2.5908" y2="17.2212" width="0.1524" layer="1"/>
 <wire x1="11.2776" y1="23.3172" x2="5.1816" y2="17.2212" width="0.1524" layer="1"/>
@@
 <signal name="ANLG2">
 <contactref element="S2R" pad="8"/>
-<contactref element="JP1" pad="11"/>
+<contactref element="SV1" pad="11"/>
 <wire x1="10.668" y1="17.2212" x2="7.62" y2="17.2212" width="0.1524" layer="1"/>
 <wire x1="11.7348" y1="18.288" x2="10.668" y2="17.2212" width="0.1524" layer="1"/>
