File: hardware/peripheral/p2rly-001.brd (EAGLE design)
At the start: 18 x 31 mm, 5 parts

Commit message: Relay port.
Parts:
- removed JP1: (no value), pinhead:2X08
- removed S1C, S2R: (no value), switch-dil:A1353HEX
- added J4: RLY, SparkFun-Connectors:JST-3-PTH-VERT
- added JRLY: AUDIO_JACK_3.5MM_KIT, SparkFun-Connectors:AUDIO-JACK-KIT
- moved U$1 17.6 mm to (6.50, 4.50), flipped to the top, turned to 0 degrees
- moved LOGO1 14.1 mm to (6.50, 24.0), turned to 0 degrees
Connections:
- removed net ANLG0: JP1.3, S2R.1
- removed net ANLG1: JP1.7, S2R.4
- removed net ANLG2: JP1.11, S2R.8
- removed net ANLG3: JP1.15, S2R.2
- removed net DTCT0: JP1.2, S1C.1
- removed net DTCT1: JP1.6, S1C.4
- removed net DTCT2: JP1.10, S1C.8
- removed net DTCT3: JP1.14, S1C.2
- removed net GND: JP1.1, JP1.13, JP1.5, JP1.9, S1C.C
- removed net VCC: JP1.12, JP1.16, JP1.4, JP1.8, S2R.C
- new net COMMON: J4.2, JRLY.SLEEVE
- new net NC: J4.3, JRLY.RING
- new net NO: J4.1, JRLY.TIP
Routing:
- net VCC: track 31.7 -> 0.00 mm
- net GND: track 28.5 -> 0.00 mm
- net DTCT3: track 20.4 -> 0.00 mm
- net ANLG0: track 19.9 -> 0.00 mm
- net ANLG1: track 16.4 -> 0.00 mm
- net DTCT2: track 15.0 -> 0.00 mm
- net ANLG3: track 14.8 -> 0.00 mm
- net NC: track 0.00 -> 12.1 mm
- net COMMON: track 0.00 -> 10.7 mm
- net DTCT1: track 10.1 -> 0.00 mm
- net NO: track 0.00 -> 9.15 mm
- net DTCT0: track 8.95 -> 0.00 mm
- net ANLG2: track 7.60 -> 0.00 mm
- removed copper zone on layer 1, net GND
- removed copper zone on layer 16, net GND
Other:
- board text added: "Avvicon MJ-495"
- board text added: "N.C."
- board text added: "N.O."
- board text added: "RLY Port 0.0.1-X"
- board text added: "Ring"
- board text added: "Sleeve"
- board text added: "Tip"
- board text removed: "A0"
- board text removed: "A1"
- board text removed: "A2"
- board text removed: "A3"
- board text removed: "D10"
- board text removed: "D12"
- board text removed: "D6"
- board text removed: "D9"
- board text removed: "G"
- board text removed: "Hex Sw 0.0.1-X"
- board text removed: "V/2"
