File: hardware/peripheral/p2rly-001.brd (EAGLE design)
At the start: 18 x 31 mm, 4 parts, among them J4 RLY

Commit message: Symbol name.
Parts:
- renumbered JRLY to JJ4
Changed lines of the file:
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@@
 <element name="LOGO1" library="SparkFun-Aesthetics" package="OSHW-LOGO-S_COPPER" value="OSHW-LOGOS-COPPER" x="6.5" y="24" smashed="yes" rot="MR0"/>
 <element name="U$1" library="pineapple" package="PINEAPPLE450_SILK" value="PINEAPPLE450_SILK" x="6.5" y="4.5" smashed="yes"/>
-<element name="JRLY" library="SparkFun-Connectors" library_urn="urn:adsk.eagle:library:513" package="AUDIO-JACK-KIT" package3d_urn="urn:adsk.eagle:package:38014/1" value="AUDIO_JACK_3.5MM_KIT" x="4.5" y="15.5" smashed="yes">
+<element name="JJ4" library="SparkFun-Connectors" library_urn="urn:adsk.eagle:library:513" package="AUDIO-JACK-KIT" package3d_urn="urn:adsk.eagle:package:38014/1" value="AUDIO_JACK_3.5MM_KIT" x="4.5" y="15.5" smashed="yes">
 <attribute name="NAME" x="3" y="22.5" size="1" layer="25" ratio="20" align="bottom-center"/>
 <attribute name="PROD_ID" value="CONN-08774" x="4.5" y="15.5" size="1.778" layer="27" display="off"/>
@@
 <signals>
 <signal name="NO">
-<contactref element="JRLY" pad="TIP"/>
+<contactref element="JJ4" pad="TIP"/>
 <contactref element="J4" pad="1"/>
 <wire x1="14.3256" y1="16.9164" x2="14.3256" y2="17.3736" width="0.1524" layer="16"/>
@@
 </signal>
 <signal name="COMMON">
-<contactref element="JRLY" pad="SLEEVE"/>
+<contactref element="JJ4" pad="SLEEVE"/>
 <contactref element="J4" pad="2"/>
 <wire x1="10.8204" y1="15.5448" x2="14.3256" y2="15.5448" width="0.1524" layer="1"/>
@@
 </signal>
 <signal name="NC">
-<contactref element="JRLY" pad="RING"/>
+<contactref element="JJ4" pad="RING"/>
 <contactref element="J4" pad="3"/>
 <wire x1="14.478" y1="14.0208" x2="14.478" y2="13.5636" width="0.1524" layer="1"/>
