File: hardware/peripheral/p2rly-001.sch (EAGLE design)
At the start: 5 parts

Commit message: Relay port.
Parts:
- removed JP1: (no value), pinhead:PINHD-2X8
- removed S1C, S2R: (no value), switch-dil:A1353HEX
- added J4: RLY, SparkFun-Connectors:CONN_03JST-PTH-VERT
- added JRLY: AUDIO_JACK_3.5MM_KIT, SparkFun-Connectors:AUDIO_JACK_3.5MM_KIT
Connections:
- removed net ANLG0: JP1.3, S2R.1
- removed net ANLG1: JP1.7, S2R.4
- removed net ANLG2: JP1.11, S2R.8
- removed net ANLG3: JP1.15, S2R.2
- removed net DTCT0: JP1.2, S1C.1
- removed net DTCT1: JP1.6, S1C.4
- removed net DTCT2: JP1.10, S1C.8
- removed net DTCT3: JP1.14, S1C.2
- removed net GND: JP1.1, JP1.13, JP1.5, JP1.9, S1C.C
- removed net VCC: JP1.12, JP1.16, JP1.4, JP1.8, S2R.C
- new net COMMON: J4.2, JRLY.SLEEVE
- new net NC: J4.3, JRLY.RING
- new net NO: J4.1, JRLY.TIP
Other:
- note removed: "GeekPort II 1: GND 2: DTCT0 3: ANLG0 4: Vcc/2"
- note removed: "Pineapple -> Switch 1->1 2->4 4->8 8->2"

Commit message: Symbol name.
Parts:
- renumbered JRLY to JJ4
Changed lines of the file:
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@@
 <part name="LOGO1" library="SparkFun-Aesthetics" deviceset="OSHW-LOGO" device="S-COPPER" value="OSHW-LOGOS-COPPER"/>
 <part name="U$1" library="pineapple" deviceset="PINEAPPLE450_SILK" device=""/>
-<part name="JRLY" library="SparkFun-Connectors" library_urn="urn:adsk.eagle:library:513" deviceset="AUDIO_JACK_3.5MM" device="_KIT" package3d_urn="urn:adsk.eagle:package:38014/1"/>
+<part name="JJ4" library="SparkFun-Connectors" library_urn="urn:adsk.eagle:library:513" deviceset="AUDIO_JACK_3.5MM" device="_KIT" package3d_urn="urn:adsk.eagle:package:38014/1"/>
 <part name="J4" library="SparkFun-Connectors" library_urn="urn:adsk.eagle:library:513" deviceset="CONN_03" device="JST-PTH-VERT" package3d_urn="urn:adsk.eagle:package:38080/1" value="RLY"/>
 </parts>
@@
 <instance part="LOGO1" gate="G$1" x="241.3" y="165.1" smashed="yes"/>
 <instance part="U$1" gate="G$1" x="241.3" y="142.24" smashed="yes"/>
-<instance part="JRLY" gate="G$1" x="30.48" y="124.46" smashed="yes">
+<instance part="JJ4" gate="G$1" x="30.48" y="124.46" smashed="yes">
 <attribute name="NAME" x="25.4" y="130.048" size="1.778" layer="95" font="vector"/>
 <attribute name="VALUE" x="25.4" y="116.84" size="1.778" layer="96" font="vector"/>
@@
 <net name="NO" class="0">
 <segment>
-<pinref part="JRLY" gate="G$1" pin="TIP"/>
+<pinref part="JJ4" gate="G$1" pin="TIP"/>
 <pinref part="J4" gate="J$1" pin="1"/>
 <wire x1="35.56" y1="119.38" x2="71.12" y2="119.38" width="0.1524" layer="91"/>
@@
 <net name="COMMON" class="0">
 <segment>
-<pinref part="JRLY" gate="G$1" pin="SLEEVE"/>
+<pinref part="JJ4" gate="G$1" pin="SLEEVE"/>
 <wire x1="35.56" y1="129.54" x2="43.18" y2="129.54" width="0.1524" layer="91"/>
 <wire x1="43.18" y1="129.54" x2="43.18" y2="121.92" width="0.1524" layer="91"/>
@@
 <net name="NC" class="0">
 <segment>
-<pinref part="JRLY" gate="G$1" pin="RING"/>
+<pinref part="JJ4" gate="G$1" pin="RING"/>
 <wire x1="35.56" y1="127" x2="45.72" y2="127" width="0.1524" layer="91"/>
 <wire x1="45.72" y1="127" x2="45.72" y2="124.46" width="0.1524" layer="91"/>
