File: hardware/peripheral/p2hex-001.sch (EAGLE design)
At the start: 5 parts

Commit message: Silk.
Parts:
- renumbered S1 to S1C, S2 to S2R
Changed lines of the file:
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@@
 <part name="LOGO1" library="SparkFun-Aesthetics" deviceset="OSHW-LOGO" device="S-COPPER" value="OSHW-LOGOS-COPPER"/>
 <part name="JP1" library="pinhead" library_urn="urn:adsk.eagle:library:325" deviceset="PINHD-2X8" device="" package3d_urn="urn:adsk.eagle:package:22481/2"/>
-<part name="S1" library="switch-dil" library_urn="urn:adsk.eagle:library:375" deviceset="A1353HEX" device="" package3d_urn="urn:adsk.eagle:package:27207/1"/>
-<part name="S2" library="switch-dil" library_urn="urn:adsk.eagle:library:375" deviceset="A1353HEX" device="" package3d_urn="urn:adsk.eagle:package:27207/1"/>
+<part name="S1C" library="switch-dil" library_urn="urn:adsk.eagle:library:375" deviceset="A1353HEX" device="" package3d_urn="urn:adsk.eagle:package:27207/1"/>
+<part name="S2R" library="switch-dil" library_urn="urn:adsk.eagle:library:375" deviceset="A1353HEX" device="" package3d_urn="urn:adsk.eagle:package:27207/1"/>
 <part name="SUPPLY1" library="supply2" library_urn="urn:adsk.eagle:library:372" deviceset="GND" device=""/>
 <part name="SUPPLY2" library="supply2" library_urn="urn:adsk.eagle:library:372" deviceset="GND" device=""/>
@@
 <attribute name="VALUE" x="105.41" y="86.36" size="1.778" layer="96"/>
 </instance>
-<instance part="S1" gate="1" x="40.64" y="101.6" smashed="yes">
+<instance part="S1C" gate="1" x="40.64" y="101.6" smashed="yes">
 <attribute name="NAME" x="36.195" y="96.52" size="1.778" layer="95" rot="R90"/>
 <attribute name="VALUE" x="49.53" y="96.52" size="1.778" layer="96" rot="R90"/>
 </instance>
-<instance part="S2" gate="1" x="60.96" y="101.6" smashed="yes" rot="R180">
+<instance part="S2R" gate="1" x="60.96" y="101.6" smashed="yes" rot="R180">
 <attribute name="NAME" x="65.405" y="106.68" size="1.778" layer="95" rot="R270"/>
 <attribute name="VALUE" x="52.07" y="106.68" size="1.778" layer="96" rot="R270"/>
@@
 </segment>
 <segment>
-<pinref part="S1" gate="1" pin="C"/>
+<pinref part="S1C" gate="1" pin="C"/>
 <wire x1="40.64" y1="93.98" x2="40.64" y2="81.28" width="0.1524" layer="91"/>
 <pinref part="SUPPLY2" gate="GND" pin="GND"/>
@@
 </segment>
 <segment>
-<pinref part="S1" gate="1" pin="1"/>
+<pinref part="S1C" gate="1" pin="1"/>
 <wire x1="38.1" y1="109.22" x2="38.1" y2="114.3" width="0.1524" layer="91"/>
 <label x="38.1" y="114.3" size="0.8128" layer="95" rot="R90" xref="yes"/>
@@
 </segment>
 <segment>
-<pinref part="S2" gate="1" pin="C"/>
+<pinref part="S2R" gate="1" pin="C"/>
 <wire x1="60.96" y1="109.22" x2="60.96" y2="114.3" width="0.1524" layer="91"/>
 <pinref part="SUPPLY4" gate="G$1" pin="VCC"/>
@@
 </segment>
 <segment>
-<pinref part="S1" gate="1" pin="4"/>
+<pinref part="S1C" gate="1" pin="4"/>
 <wire x1="43.18" y1="109.22" x2="43.18" y2="114.3" width="0.1524" layer="91"/>
 <label x="43.18" y="114.3" size="0.8128" layer="95" rot="R90" xref="yes"/>
@@
 </segment>
 <segment>
-<pinref part="S1" gate="1" pin="8"/>
+<pinref part="S1C" gate="1" pin="8"/>
 <wire x1="45.72" y1="109.22" x2="45.72" y2="114.3" width="0.1524" layer="91"/>
 <label x="45.72" y="114.3" size="0.8128" layer="95" rot="R90" xref="yes"/>
@@
 </segment>
 <segment>
-<pinref part="S1" gate="1" pin="2"/>
+<pinref part="S1C" gate="1" pin="2"/>
 <wire x1="40.64" y1="109.22" x2="40.64" y2="114.3" width="0.1524" layer="91"/>
 <label x="40.64" y="114.3" size="0.8128" layer="95" rot="R90" xref="yes"/>
@@
 </segment>
 <segment>
-<pinref part="S2" gate="1" pin="1"/>
+<pinref part="S2R" gate="1" pin="1"/>
 <wire x1="63.5" y1="93.98" x2="63.5" y2="88.9" width="0.1524" layer="91"/>
 <label x="63.5" y="88.9" size="0.8128" layer="95" rot="R270" xref="yes"/>
@@
 </segment>
 <segment>
-<pinref part="S2" gate="1" pin="4"/>
+<pinref part="S2R" gate="1" pin="4"/>
 <wire x1="58.42" y1="93.98" x2="58.42" y2="88.9" width="0.1524" layer="91"/>
 <label x="58.42" y="88.9" size="0.8128" layer="95" rot="R270" xref="yes"/>
@@
 <net name="ANLG3" class="0">
 <segment>
-<pinref part="S2" gate="1" pin="2"/>
+<pinref part="S2R" gate="1" pin="2"/>
 <wire x1="60.96" y1="93.98" x2="60.96" y2="88.9" width="0.1524" layer="91"/>
 <label x="60.96" y="88.9" size="0.8128" layer="95" rot="R270" xref="yes"/>
@@
 <net name="ANLG2" class="0">
 <segment>
-<pinref part="S2" gate="1" pin="8"/>
+<pinref part="S2R" gate="1" pin="8"/>
 <wire x1="55.88" y1="93.98" x2="55.88" y2="88.9" width="0.1524" layer="91"/>
 <label x="55.88" y="88.9" size="0.8128" layer="95" rot="R270" xref="yes"/>

Commit message: Silk.
Parts:
- renumbered JP1 to SV1
Changed lines of the file:
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@@
 <part name="FRAME1" library="frames" library_urn="urn:adsk.eagle:library:229" deviceset="A4L-LOC" device=""/>
 <part name="LOGO1" library="SparkFun-Aesthetics" deviceset="OSHW-LOGO" device="S-COPPER" value="OSHW-LOGOS-COPPER"/>
-<part name="JP1" library="pinhead" library_urn="urn:adsk.eagle:library:325" deviceset="PINHD-2X8" device="" package3d_urn="urn:adsk.eagle:package:22481/2"/>
+<part name="SV1" library="pinhead" library_urn="urn:adsk.eagle:library:325" deviceset="PINHD-2X8" device="" package3d_urn="urn:adsk.eagle:package:22481/2"/>
 <part name="S1C" library="switch-dil" library_urn="urn:adsk.eagle:library:375" deviceset="A1353HEX" device="" package3d_urn="urn:adsk.eagle:package:27207/1"/>
 <part name="S2R" library="switch-dil" library_urn="urn:adsk.eagle:library:375" deviceset="A1353HEX" device="" package3d_urn="urn:adsk.eagle:package:27207/1"/>
@@
 </instance>
 <instance part="LOGO1" gate="G$1" x="241.3" y="165.1" smashed="yes"/>
-<instance part="JP1" gate="A" x="111.76" y="101.6" smashed="yes">
+<instance part="SV1" gate="A" x="111.76" y="101.6" smashed="yes">
 <attribute name="NAME" x="105.41" y="112.395" size="1.778" layer="95"/>
 <attribute name="VALUE" x="105.41" y="86.36" size="1.778" layer="96"/>
@@
 <net name="GND" class="0">
 <segment>
-<pinref part="JP1" gate="A" pin="1"/>
+<pinref part="SV1" gate="A" pin="1"/>
 <wire x1="109.22" y1="109.22" x2="101.6" y2="109.22" width="0.1524" layer="91"/>
 <wire x1="101.6" y1="109.22" x2="101.6" y2="104.14" width="0.1524" layer="91"/>
 <pinref part="SUPPLY1" gate="GND" pin="GND"/>
-<pinref part="JP1" gate="A" pin="5"/>
+<pinref part="SV1" gate="A" pin="5"/>
 <wire x1="101.6" y1="104.14" x2="101.6" y2="99.06" width="0.1524" layer="91"/>
 <wire x1="101.6" y1="99.06" x2="101.6" y2="93.98" width="0.1524" layer="91"/>
@@
 <wire x1="109.22" y1="104.14" x2="101.6" y2="104.14" width="0.1524" layer="91"/>
 <junction x="101.6" y="104.14"/>
-<pinref part="JP1" gate="A" pin="9"/>
+<pinref part="SV1" gate="A" pin="9"/>
 <wire x1="109.22" y1="99.06" x2="101.6" y2="99.06" width="0.1524" layer="91"/>
 <junction x="101.6" y="99.06"/>
-<pinref part="JP1" gate="A" pin="13"/>
+<pinref part="SV1" gate="A" pin="13"/>
 <wire x1="109.22" y1="93.98" x2="101.6" y2="93.98" width="0.1524" layer="91"/>
 <junction x="101.6" y="93.98"/>
@@
 <net name="DTCT0" class="0">
 <segment>
-<pinref part="JP1" gate="A" pin="2"/>
+<pinref part="SV1" gate="A" pin="2"/>
 <wire x1="116.84" y1="109.22" x2="132.08" y2="109.22" width="0.1524" layer="91"/>
 <label x="132.08" y="109.22" size="0.8128" layer="95" xref="yes"/>
@@
 <net name="VCC" class="0">
 <segment>
-<pinref part="JP1" gate="A" pin="4"/>
+<pinref part="SV1" gate="A" pin="4"/>
 <wire x1="116.84" y1="106.68" x2="124.46" y2="106.68" width="0.1524" layer="91"/>
 <wire x1="124.46" y1="106.68" x2="124.46" y2="124.46" width="0.1524" layer="91"/>
 <pinref part="SUPPLY3" gate="G$1" pin="VCC"/>
-<pinref part="JP1" gate="A" pin="16"/>
+<pinref part="SV1" gate="A" pin="16"/>
 <wire x1="116.84" y1="91.44" x2="124.46" y2="91.44" width="0.1524" layer="91"/>
 <wire x1="124.46" y1="91.44" x2="124.46" y2="96.52" width="0.1524" layer="91"/>
 <junction x="124.46" y="106.68"/>
-<pinref part="JP1" gate="A" pin="12"/>
+<pinref part="SV1" gate="A" pin="12"/>
 <wire x1="124.46" y1="96.52" x2="124.46" y2="101.6" width="0.1524" layer="91"/>
 <wire x1="124.46" y1="101.6" x2="124.46" y2="106.68" width="0.1524" layer="91"/>
 <wire x1="116.84" y1="96.52" x2="124.46" y2="96.52" width="0.1524" layer="91"/>
 <junction x="124.46" y="96.52"/>
-<pinref part="JP1" gate="A" pin="8"/>
+<pinref part="SV1" gate="A" pin="8"/>
 <wire x1="116.84" y1="101.6" x2="124.46" y2="101.6" width="0.1524" layer="91"/>
 <junction x="124.46" y="101.6"/>
@@
 <net name="DTCT1" class="0">
 <segment>
-<pinref part="JP1" gate="A" pin="6"/>
+<pinref part="SV1" gate="A" pin="6"/>
 <wire x1="116.84" y1="104.14" x2="132.08" y2="104.14" width="0.1524" layer="91"/>
 <label x="132.08" y="104.14" size="0.8128" layer="95" xref="yes"/>
@@
 <net name="DTCT2" class="0">
 <segment>
-<pinref part="JP1" gate="A" pin="10"/>
+<pinref part="SV1" gate="A" pin="10"/>
 <wire x1="116.84" y1="99.06" x2="132.08" y2="99.06" width="0.1524" layer="91"/>
 <label x="132.08" y="99.06" size="0.8128" layer="95" xref="yes"/>
@@
 <net name="DTCT3" class="0">
 <segment>
-<pinref part="JP1" gate="A" pin="14"/>
+<pinref part="SV1" gate="A" pin="14"/>
 <wire x1="116.84" y1="93.98" x2="132.08" y2="93.98" width="0.1524" layer="91"/>
 <label x="132.08" y="93.98" size="0.8128" layer="95" xref="yes"/>
@@
 <net name="ANLG0" class="0">
 <segment>
-<pinref part="JP1" gate="A" pin="3"/>
+<pinref part="SV1" gate="A" pin="3"/>
 <wire x1="109.22" y1="106.68" x2="96.52" y2="106.68" width="0.1524" layer="91"/>
 <label x="96.52" y="106.68" size="0.8128" layer="95" rot="R180" xref="yes"/>
@@
 <net name="ANLG1" class="0">
 <segment>
-<pinref part="JP1" gate="A" pin="7"/>
+<pinref part="SV1" gate="A" pin="7"/>
 <wire x1="109.22" y1="101.6" x2="96.52" y2="101.6" width="0.1524" layer="91"/>
 <label x="96.52" y="101.6" size="0.8128" layer="95" rot="R180" xref="yes"/>
@@
 </segment>
 <segment>
-<pinref part="JP1" gate="A" pin="15"/>
+<pinref part="SV1" gate="A" pin="15"/>
 <wire x1="109.22" y1="91.44" x2="96.52" y2="91.44" width="0.1524" layer="91"/>
 <label x="96.52" y="91.44" size="0.8128" layer="95" rot="R180" xref="yes"/>
@@
 </segment>
 <segment>
-<pinref part="JP1" gate="A" pin="11"/>
+<pinref part="SV1" gate="A" pin="11"/>
 <wire x1="109.22" y1="96.52" x2="96.52" y2="96.52" width="0.1524" layer="91"/>
 <label x="96.52" y="96.52" size="0.8128" layer="95" rot="R180" xref="yes"/>
